File: bspd-kicad/bspd.kicad_sch (KiCad schematic)
At the start: 52 parts, among them J1 BSPD Connector, Q1 AO3400A, U1 MCP1703T-5002E/CB, U6 SN74LVC3G14DCUR, U7 SN74LVC2G00DCTR

Commit message: Switched to D latch chip
Parts:
- removed U6: SN74LVC3G14DCUR, bspd:SN74LVC3G14DCUR, symbol bspd:SN74LVC3G14DCUR
- removed U7: SN74LVC2G00DCTR, bspd:SN74LVC2G00DCTR, symbol bspd:SN74LVC2G00DCTR
- added U7: SN74LVC2G14DBVR, bspd:SN74LVC2G14DBVR, symbol bspd:SN74LVC2G14DBVR
- added U8: 74HC74, Package_SO:SOIC-14-16_3.9x9.9mm_P1.27mm, symbol 74xx:74HC74
- C10: value xuF -> 2.2uF
- R29: value x -> 330k
Connections:
- net +5V: now also U7.5 (VCC)
- net Earth: now also U7.2 (GND), U8.2 (D), U8.3 (C)
- net FAULT: now also U8.4 (~{S})
- net at C10.1, D4.2 (A), R29.1: now also U7.1
- net at Q1.1 (G): now also U8.5 (Q)
- new net: U7.4, U8.1 (~{R})
- new net: U7.3, U7.6
- no-connect marks 0 -> 1
Other:
- note added: "SR Latch"
- note added: "TODO: Measure Shutdown circuit current, its probs ~200mA Check if BSPD currently uses Chassis GND or Signal GND If Chassis, impliment comparator"
- note added: "~R"
- note added: "~S"
- note removed: "Inverting to FAULT HIGH logic"
- note removed: "R"
- note removed: "S"
- note removed: "SR Latch, Cross Coupled NAND"
- moved on the sheet: C10, D4, R29
