File: bspd-kicad/bspd.kicad_pcb (KiCad board)
At the start: 2 copper layers, 100 x 80 mm, 107 parts, among them Q1 AO3401A, Q2 AO3400A, SW1 CJS-1200TB1, SW2 CJS-1200TB1, U10 LM1117MP-5.0, U5 SN74HC74DR, U7 SN74LVC2G14DBVR, U8 SN74LVC3G14DCUR, U9 SN74LVC3G14DCUR

Commit message: Layout Progress
Parts:
- removed the D14 at (68.2, 43.0)
- added D7: S1B-13-F, bspd:S1B-13-F, F.Cu at (69.2, 39.7)
- added D8: S1B-13-F, bspd:S1B-13-F, F.Cu at (69.2, 44.2)
- added R34: 10M, Resistor_SMD:R_0805_2012Metric_Pad1.20x1.40mm_HandSolder, F.Cu at (40.4, 64.0)
- added R35: 10M, Resistor_SMD:R_0805_2012Metric_Pad1.20x1.40mm_HandSolder, F.Cu at (40.4, 67.0)
- added R36: 10M, Resistor_SMD:R_0805_2012Metric_Pad1.20x1.40mm_HandSolder, F.Cu at (40.4, 70.0)
- added R37: 10M, Resistor_SMD:R_0805_2012Metric_Pad1.20x1.40mm_HandSolder, F.Cu at (40.4, 72.9)
- added R38: 10M, Resistor_SMD:R_0805_2012Metric_Pad1.20x1.40mm_HandSolder, F.Cu at (40.4, 75.8)
- R24: value 4.99k -> 2.61k
- R28: value 45.3k -> 49.9k
- moved C12 6.83 mm to (54.5, 64.2)
- moved C13 6.83 mm to (44.7, 64.2)
- moved C14 6.83 mm to (49.7, 64.2)
- moved C17 6.83 mm to (59.4, 64.2)
- moved C18 6.83 mm to (64.4, 64.2)
- moved RV1 6.83 mm to (44.6, 68.2)
- moved RV2 6.83 mm to (49.5, 68.2)
- moved RV3 6.83 mm to (54.5, 68.2)
- moved RV4 6.83 mm to (59.4, 68.2)
- moved RV5 6.83 mm to (64.4, 68.2)
- moved SW1 6.83 mm to (71.3, 66.3)
- moved SW2 6.83 mm to (71.6, 73.5)
- moved C25 2.03 mm to (105.0, 39.0)
- moved C10 1.25 mm to (62.7, 26.0)
- moved C11 1.25 mm to (70.2, 26.0)
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- renumbered C27 to C10, C28 to C11, C23 to C12, C21 to C13, C22 to C14, C8 to C15, C9 to C16, C20 to C17, C24 to C18, C10 to C20, C11 to C21, C12 to C22, C13 to C23, C14 to C24, C15 to C25, C16 to C26, C17 to C27, C18 to C28, C25 to C8, C26 to C9, D8 to D10, D9 to D11, D10 to D12, D11 to D13, D12 to D14, D13 to D15, D6 to D5, D5 to D6, D7 to D9, Q2 to Q1, Q1 to Q2, R39 to R29, R40 to R30, R29 to R31, R30 to R32, R31 to R33, R32 to R39, R33 to R40, R34 to R41, R35 to R42, R36 to R43, R37 to R44, R38 to R45, U4 to U2, U2 to U4, U10 to U6
Connections:
- net +4V5 renamed +4V7
- Q1 pad 1: Net-(Q2-G) (its old number) -> OUTPUT
- R31 pad 2: Net-(Q2-G) (its old number) -> OUTPUT
- R33 pad 2: Net-(Q2-G) (its old number) -> OUTPUT
