File: bspd-kicad/bspd.kicad_pcb (KiCad board)
At the start: 4 copper layers, 75.5 x 62 mm, 121 parts, among them J1 Conn_02x04_Counter_Clockwise, Q1 AO3400A, Q2 AO3401A, SW1 CJS-1200TB1, SW2 CJS-1200TB1, U1 TLV1704AIPWR, U2 TLV1704AIPWR, U3 TLV1704AIPWR, U4 TLV1704AIPWR, U5 SN74HC74DR, U6 LM1117MP-5.0, U7 SN74LVC2G14DBVR, U8 SN74LVC3G14DCUR, U9 SN74LVC3G14DCUR

Commit message: update
Other:
- board text added: "4.7V"
- board text removed: "4.5V"
Changed lines of the file:
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@@
 		)
 	)
-	(gr_text "4.5V"
+	(gr_text "4.7V"
 		(at 62.016584 132.945588 0)
 		(layer "F.SilkS")

Commit message: Signal ground and chassis ground connected with 0 ohm resistor
Parts:
- added R46: 0, Resistor_SMD:R_0805_2012Metric_Pad1.20x1.40mm_HandSolder, F.Cu at (27.0, 126.0)
- moved D2 0.40 mm to (27.1, 111.8)
- moved D3 0.26 mm to (35.8, 111.8)
Connections:
- J1 pad 4: GND -> /SENS_0V
Routing:
- net GND: track 97.8 -> 101.0 mm, vias 329 -> 333
- net /SENS_0V: track 0.00 -> 3.21 mm
- net +5V: track 78.1 -> 79.1 mm, vias 35 -> 36
- net +12V: vias 4 -> 5

Commit message: Fix mislabeled RV1-RV5 trimmer footprint and remove unused duplicate diode footprint
The trimpot footprint was named/described as a 10k part when it's actually the 20k version used on the board; renamed it to match. Also removed a custom TVS diode footprint that was never used since D2-D4 already used KiCad's built-in equivalent footprint.
Parts:
- RV1, RV2, RV3, RV4, RV5: footprint bspd:3313J-1-103E -> bspd:3313J-1-203E
Changed lines of the file:
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@@
 		)
 	)
-	(footprint "bspd:3313J-1-103E"
+	(footprint "bspd:3313J-1-203E"
 		(layer "F.Cu")
 		(at 72.783604 137.684024)
-		(descr "Bourns 3313J-1-103E, 3mm square single-turn cermet SMD trimmer potentiometer, 10k ohm, top adjust. Land pattern per Bourns 3313 datasheet (3313J style). https://www.bourns.com/docs/Product-Datasheets/3313.pdf")
+		(descr "Bourns 3313J-1-203E, 3mm square single-turn cermet SMD trimmer potentiometer, 10k ohm, top adjust. Land pattern per Bourns 3313 datasheet (3313J style). https://www.bourns.com/docs/Product-Datasheets/3313.pdf")
 		(tags "trimmer potentiometer trimpot Bourns 3313 3313J SMD 10k")
 		(property "Reference" "RV2"
@@
 		)
 		(embedded_fonts no)
-		(model "${KIPRJMOD}/bspd-library/3d/3313J-1-103E.step"
+		(model "${KIPRJMOD}/bspd-library/3d/3313J-1-203E.step"
 			(offset
 				(xyz 0 0 0)
@@
 		)
 	)
-	(footprint "bspd:3313J-1-103E"
+	(footprint "bspd:3313J-1-203E"
 		(layer "F.Cu")
 		(at 77.733604 137.684024)
-		(descr "Bourns 3313J-1-103E, 3mm square single-turn cermet SMD trimmer potentiometer, 10k ohm, top adjust. Land pattern per Bourns 3313 datasheet (3313J style). https://www.bourns.com/docs/Product-Datasheets/3313.pdf")
+		(descr "Bourns 3313J-1-203E, 3mm square single-turn cermet SMD trimmer potentiometer, 10k ohm, top adjust. Land pattern per Bourns 3313 datasheet (3313J style). https://www.bourns.com/docs/Product-Datasheets/3313.pdf")
 		(tags "trimmer potentiometer trimpot Bourns 3313 3313J SMD 10k")
 		(property "Reference" "RV3"
@@
 		)
 		(embedded_fonts no)
-		(model "${KIPRJMOD}/bspd-library/3d/3313J-1-103E.step"
+		(model "${KIPRJMOD}/bspd-library/3d/3313J-1-203E.step"
 			(offset
 				(xyz 0 0 0)
@@
 		)
 	)
-	(footprint "bspd:3313J-1-103E"
+	(footprint "bspd:3313J-1-203E"
 		(layer "F.Cu")
 		(at 87.608604 137.684024)
-		(descr "Bourns 3313J-1-103E, 3mm square single-turn cermet SMD trimmer potentiometer, 10k ohm, top adjust. Land pattern per Bourns 3313 datasheet (3313J style). https://www.bourns.com/docs/Product-Datasheets/3313.pdf")
+		(descr "Bourns 3313J-1-203E, 3mm square single-turn cermet SMD trimmer potentiometer, 10k ohm, top adjust. Land pattern per Bourns 3313 datasheet (3313J style). https://www.bourns.com/docs/Product-Datasheets/3313.pdf")
 		(tags "trimmer potentiometer trimpot Bourns 3313 3313J SMD 10k")
 		(property "Reference" "RV5"
@@
 		)
 		(embedded_fonts no)
-		(model "${KIPRJMOD}/bspd-library/3d/3313J-1-103E.step"
+		(model "${KIPRJMOD}/bspd-library/3d/3313J-1-203E.step"
 			(offset
 				(xyz 0 0 0)
@@
 		)
 	)
-	(footprint "bspd:3313J-1-103E"
+	(footprint "bspd:3313J-1-203E"
 		(layer "F.Cu")
 		(at 82.658604 137.684024)
-		(descr "Bourns 3313J-1-103E, 3mm square single-turn cermet SMD trimmer potentiometer, 10k ohm, top adjust. Land pattern per Bourns 3313 datasheet (3313J style). https://www.bourns.com/docs/Product-Datasheets/3313.pdf")
+		(descr "Bourns 3313J-1-203E, 3mm square single-turn cermet SMD trimmer potentiometer, 10k ohm, top adjust. Land pattern per Bourns 3313 datasheet (3313J style). https://www.bourns.com/docs/Product-Datasheets/3313.pdf")
 		(tags "trimmer potentiometer trimpot Bourns 3313 3313J SMD 10k")
 		(property "Reference" "RV4"
@@
 		)
 		(embedded_fonts no)
-		(model "${KIPRJMOD}/bspd-library/3d/3313J-1-103E.step"
+		(model "${KIPRJMOD}/bspd-library/3d/3313J-1-203E.step"
 			(offset
 				(xyz 0 0 0)
@@
 		)
 	)
-	(footprint "bspd:3313J-1-103E"
+	(footprint "bspd:3313J-1-203E"
 		(layer "F.Cu")
 		(at 67.833604 137.684024)
-		(descr "Bourns 3313J-1-103E, 3mm square single-turn cermet SMD trimmer potentiometer, 10k ohm, top adjust. Land pattern per Bourns 3313 datasheet (3313J style). https://www.bourns.com/docs/Product-Datasheets/3313.pdf")
+		(descr "Bourns 3313J-1-203E, 3mm square single-turn cermet SMD trimmer potentiometer, 10k ohm, top adjust. Land pattern per Bourns 3313 datasheet (3313J style). https://www.bourns.com/docs/Product-Datasheets/3313.pdf")
 		(tags "trimmer potentiometer trimpot Bourns 3313 3313J SMD 10k")
 		(property "Reference" "RV1"
@@
 		)
 		(embedded_fonts no)
-		(model "${KIPRJMOD}/bspd-library/3d/3313J-1-103E.step"
+		(model "${KIPRJMOD}/bspd-library/3d/3313J-1-203E.step"
 			(offset
 				(xyz 0 0 0)
